Commit message: update

File: bumperbot_ws/install/bumperbot_description/share/bumperbot_description/urdf/bumperbot_gazebo.xacro (robot description, xacro)
@@ -25,4 +25,5 @@
     <maxVel>0.1</maxVel>
     <fdir1>1 0 0</fdir1>
+    <material>Gazebo/Blue</material>
   </gazebo>
   <gazebo reference="wheel_right_link">
@@ -34,4 +35,8 @@
     <maxVel>0.1</maxVel>
     <fdir1>1 0 0</fdir1>
+    <material>Gazebo/Blue</material>
+  </gazebo>
+  <gazebo reference="base_link">
+    <material>Gazebo/Red</material>
   </gazebo>
   <!-- Caster Wheels -->
@@ -43,4 +48,5 @@
     <minDepth>0.001</minDepth>
     <maxVel>1.0</maxVel>
+    <material>Gazebo/Yellow</material>
   </gazebo>
   <gazebo reference="caster_front_link">
@@ -51,4 +57,5 @@
     <minDepth>0.001</minDepth>
     <maxVel>1.0</maxVel>
+    <material>Gazebo/Yellow</material>
   </gazebo>
   <!-- ROS 2 Control -->
